File: project_02/etch_a_sketc.sch (EAGLE design)
At the start: 13 parts, among them U1 POCKETBEAGLE

Commit message: PowerPoint and Frame Info
Other:
- note added: "Mert Culcu"
Changed lines of the file:
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@@
 <drawing>
 <settings>
-<setting alwaysvectorfont="no"/>
+<setting alwaysvectorfont="yes"/>
 <setting verticaltext="up"/>
 </settings>
@@
 <text x="190.5" y="127" size="1.778" layer="91">LEDS
 </text>
+<text x="345.44" y="20.32" size="1.778" layer="91">Mert Culcu</text>
 </plain>
 <instances>
